Commit message: hardware control added.

File: arm_description/description/gazebo_control.xacro (robot description, xacro)
@@ -7,6 +7,9 @@
     </gazebo>
     <ros2_control name="GazeboSystem" type="system">
+        <!-- <hardware>
+            <plugin>gazebo_ros2_control/GazeboSystem</plugin>
+        </hardware> -->
         <hardware>
-            <plugin>gazebo_ros2_control/GazeboSystem</plugin>
+            <plugin>dofbot_hardware/DofbotSystemHardware</plugin>
         </hardware>
         <joint name="link_1_joint">

File: arm_moveit_config/config/robot.ros2_control.xacro (robot description, xacro)
@@ -2,8 +2,7 @@
 <robot xmlns:xacro="http://www.ros.org/wiki/xacro">
     <xacro:macro name="robot_ros2_control" params="name initial_positions_file">
-        <xacro:property name="initial_positions" value="${load_yaml(initial_positions_file)['initial_positions']}"/>
+        <xacro:property name="initial_positions" value="${xacro.load_yaml(initial_positions_file)['initial_positions']}"/>
         <ros2_control name="${name}" type="system">
             <hardware>
-                <!-- By default, set up controllers for simulation. This won't work on real hardware -->
                 <plugin>mock_components/GenericSystem</plugin>
             </hardware>
