Commit message: added moveit config

File: arm_description/description/arm.xacro (robot description, xacro)
@@ -46,5 +46,17 @@
             <material name="green"/>
         </visual>
-    </link>
+        <collision>
+            <origin xyz="0 0 -0.0655" rpy="0 0 0" />
+            <geometry>
+                <cylinder radius="0.040" length="0.077"/>
+            </geometry>
+        </collision>
+        <xacro:inertial_cylinder mass="50" radius="0.040" length="0.077" >
+            <origin xyz="0 0 -0.0655" />
+        </xacro:inertial_cylinder>
+    </link>
+    <gazebo reference="base_cylinder">
+        <material>Gazebo/Green</material>
+    </gazebo>
     <!-- link 1 -->
     <joint name="link_1_joint" type="revolute">
@@ -63,5 +75,17 @@
             <material name="blue"/>
         </visual>
-    </link>
+        <collision>
+            <origin xyz="0 0 -0.0215" rpy="0 0 0" />
+            <geometry>
+                <box size="0.021 0.0415 0.011"/>
+            </geometry>
+        </collision>
+        <xacro:inertial_box mass="0.05" x="0.021" y="0.0415" z="0.011" >
+            <origin xyz="0 0 -0.0215" />
+        </xacro:inertial_box>
+    </link>
+    <gazebo reference="link_1">
+        <material>Gazebo/Blue</material>
+    </gazebo>
     <!-- link 2 -->
     <joint name="link_2_joint" type="revolute">
@@ -80,5 +104,17 @@
             <material name="blue"/>
         </visual>
-    </link>
+        <collision>
+            <origin xyz="0.02875 0 0" rpy="${pi/2} 0 -${pi/2}" />
+            <geometry>
+                <box size="0.021 0.0415 0.0785"/>
+            </geometry>
+        </collision>
+        <xacro:inertial_box mass="0.05" x="0.021" y="0.0415" z="0.0785" >
+            <origin xyz="0.02875 0 0" rpy="${pi/2} 0 -${pi/2}" />
+        </xacro:inertial_box>
+    </link>
+    <gazebo reference="link_2">
+        <material>Gazebo/Blue</material>
+    </gazebo>
     <!-- link 3 -->
     <joint name="link_3_joint" type="revolute">
@@ -97,5 +133,17 @@
             <material name="blue"/>
         </visual>
-    </link>
+        <collision>
+            <origin xyz="0.02775 0 0" rpy="${pi/2} 0 -${pi/2}" />
+            <geometry>
+                <box size="0.021 0.0415 0.0765"/>
+            </geometry>
+        </collision>
+        <xacro:inertial_box mass="0.05" x="0.021" y="0.0415" z="0.0765" >
+            <origin xyz="0.02775 0 0" rpy="${pi/2} 0 -${pi/2}" />
+        </xacro:inertial_box>
+    </link>
+    <gazebo reference="link_3">
+        <material>Gazebo/Blue</material>
+    </gazebo>
     <!-- link 4 -->
     <joint name="link_4_joint" type="revolute">
@@ -114,5 +162,17 @@
             <material name="blue"/>
         </visual>
-    </link>
+        <collision>
+            <origin xyz="0.03175 0 0" rpy="${pi/2} 0 -${pi/2}" />
+            <geometry>
+                <box size="0.021 0.0415 0.0845"/>
+            </geometry>
+        </collision>
+        <xacro:inertial_box mass="0.05" x="0.021" y="0.0415" z="0.0845" >
+            <origin xyz="0.03175 0 0" rpy="${pi/2} 0 -${pi/2}" />
+        </xacro:inertial_box>
+    </link>
+    <gazebo reference="link_4">
+        <material>Gazebo/Blue</material>
+    </gazebo>
     <!-- EEpin -->
     <joint name="ee_pin_joint" type="fixed">
@@ -130,5 +190,17 @@
             <material name="white"/>
         </visual>
-    </link>
+        <collision>
+            <origin xyz="0 0 -0.006" rpy="0 0 0" />
+            <geometry>
+                <box size="0.001 0.001 0.012"/>
+            </geometry>
+        </collision>
+        <xacro:inertial_box mass="0.001" x="0.001" y="0.001" z="0.012" >
+            <origin xyz="0 0 -0.006" rpy="0 0 0" />
+        </xacro:inertial_box>
+    </link>
+    <gazebo reference="ee_pin">
+        <material>Gazebo/White</material>
+    </gazebo>
     <!-- left-finger -->
     <!-- <joint name="left_finger_joint" type="prismatic">

File: arm_description/description/bot.urdf.xacro (robot description, xacro)
@@ -4,5 +4,5 @@
     <!-- <link name="base_link">    </link>     -->
     <xacro:include filename="arm.xacro" />
-    <!-- <xacro:include filename="gazebo_control.xacro" /> -->
+    <xacro:include filename="gazebo_control.xacro" />
     <!-- <xacro:include filename="lidar.xacro" /> -->
 <!--  -->

Commit message: all update with memory working and having support for different providers with the changed arduino code

File: arm_description/description/arm.xacro (robot description, xacro)
@@ -46,4 +46,14 @@
             <material name="green"/>
         </visual>
+        <collision>
+            <origin xyz="0 0 -0.0655" rpy="0 0 0" />
+            <geometry>
+                <cylinder radius="0.040" length="0.077"/>
+            </geometry>
+            <material name="green"/>
+        </collision>
+        <xacro:inertial_cylinder mass="0.1" radius="0.040" length="0.077">
+            <origin xyz="0 0 -0.0655" rpy="0 0 0" />
+        </xacro:inertial_cylinder>
     </link>
     <!-- link 1 -->
@@ -63,4 +73,14 @@
             <material name="blue"/>
         </visual>
+        <collision>
+            <origin xyz="0 0 -0.0215" rpy="0 0 0" />
+            <geometry>
+                <box size="0.021 0.0415 0.011"/>
+            </geometry>
+            <material name="blue"/>
+        </collision>
+        <xacro:inertial_box mass="0.1" x="0.021" y="0.0415" z="0.011">
+            <origin xyz="0 0 -0.0215" rpy="0 0 0" />
+        </xacro:inertial_box>
     </link>
     <!-- link 2 -->
@@ -80,4 +100,14 @@
             <material name="blue"/>
         </visual>
+        <collision>
+            <origin xyz="0.02875 0 0" rpy="${pi/2} 0 -${pi/2}" />
+            <geometry>
+                <box size="0.021 0.0415 0.0785"/>
+            </geometry>
+            <material name="blue"/>
+        </collision>
+        <xacro:inertial_box mass="0.1" x="0.021" y="0.0415" z="0.0785">
+            <origin xyz="0.02875 0 0" rpy="${pi/2} 0 -${pi/2}" />
+        </xacro:inertial_box>
     </link>
     <!-- link 3 -->
@@ -97,4 +127,14 @@
             <material name="blue"/>
         </visual>
+        <collision>
+            <origin xyz="0.02775 0 0" rpy="${pi/2} 0 -${pi/2}" />
+            <geometry>
+                <box size="0.021 0.0415 0.0765"/>
+            </geometry>
+            <material name="blue"/>
+        </collision>
+        <xacro:inertial_box mass="0.1" x="0.021" y="0.0415" z="0.0765">
+            <origin xyz="0.02775 0 0" rpy="${pi/2} 0 -${pi/2}" />
+        </xacro:inertial_box>
     </link>
     <!-- link 4 -->
@@ -114,4 +154,14 @@
             <material name="blue"/>
         </visual>
+        <collision>
+            <origin xyz="0.03175 0 0" rpy="${pi/2} 0 -${pi/2}" />
+            <geometry>
+                <box size="0.021 0.0415 0.0845"/>
+            </geometry>
+            <material name="blue"/>
+        </collision>
+        <xacro:inertial_box mass="0.1" x="0.021" y="0.0415" z="0.0845">
+            <origin xyz="0.03175 0 0" rpy="${pi/2} 0 -${pi/2}" />
+        </xacro:inertial_box>
     </link>
     <!-- EEpin -->
@@ -130,4 +180,14 @@
             <material name="white"/>
         </visual>
+        <collision>
+            <origin xyz="0 0 -0.006" rpy="0 0 0" />
+            <geometry>
+                <box size="0.001 0.001 0.012"/>
+            </geometry>
+            <material name="white"/>
+        </collision>
+        <xacro:inertial_box mass="0.1" x="0.001" y="0.001" z="0.012">
+            <origin xyz="0 0 -0.006" rpy="0 0 0" />
+        </xacro:inertial_box>
     </link>
     <!-- left-finger -->
@@ -147,4 +207,14 @@
             <material name="blue"/>
         </visual>
+        <collision>
+            <origin xyz="0 0 0" rpy="0 0 0" />
+            <geometry>
+                <box size="0.022 0.011 0.040"/>
+            </geometry>
+            <material name="blue"/>
+        </collision>
+        <xacro:inertial_box mass="0.1" x="0.022" y="0.011" z="0.040">
+            <origin xyz="0 0 0" rpy="0 0 0" />
+        </xacro:inertial_box>
     </link> -->
     <!-- right-finger -->
@@ -165,4 +235,14 @@
             <material name="blue"/>
         </visual>
+        <collision>
+            <origin xyz="0 0 0" rpy="0 0 0" />
+            <geometry>
+                <box size="0.022 0.011 0.040"/>
+            </geometry>
+            <material name="blue"/>
+        </collision>
+        <xacro:inertial_box mass="0.1" x="0.022" y="0.011" z="0.040">
+            <origin xyz="0 0 0" rpy="0 0 0" />
+        </xacro:inertial_box>
     </link> -->
 </robot>
